File: pcb/ocdmk.kicad_pcb (KiCad board)
At the start: 2 copper layers, 147.6 x 103.5 mm, 99 parts, among them J1 USB_C_Receptacle_USB2.0_16P, J3 Conn_ARM_SWD_TagConnect_TC203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, J4 USB_C_Receptacle_USB2.0_16P, J5 Conn_01x02_Pin, U2 MDBT50-512K, U3 MCP1662-xOT

Commit message: half completed
Parts:
- removed C2: 100n, Capacitor_SMD:C_0603_1608Metric
- removed R1: 10k, Resistor_SMD:R_0603_1608Metric
- C11: footprint Capacitor_SMD:C_0603_1608Metric -> Capacitor_SMD:C_1206_3216Metric
- J1, J4: footprint ocdmk:USB4510-03-1-A_GCT -> ocdmk:12402012E212A_AMP
- J3: footprint Connector:Tag-Connect_TC2030-IDC-NL_2x03_P1.27mm_Vertical -> Connector:Tag-Connect_TC2030-IDC-FP_2x03_P1.27mm_Vertical
- J5: footprint Connector_JST:JST_PH_S2B-PH-SM4-TB_1x02-1MP_P2.00mm_Horizontal -> Connector_JST:JST_PH_S2B-PH-K_1x02_P2.00mm_Horizontal
- JP1: footprint Resistor_SMD:R_0603_1608Metric -> Jumper:SolderJumper-2_P1.3mm_Open_TrianglePad1.0x1.5mm
- L3: value 4u7 -> 10u
- U1: value ~ -> bq25185
- moved C5 4.50 mm to (253.5, 174.0)
- moved J3 2.73 mm to (255.3, 168.1), turned to 0 degrees
- moved J5 1.45 mm to (193.8, 175.9)
- moved JP1 1.10 mm to (257.0, 174.5)
- moved C3 0.98 mm to (257.0, 178.0)
- moved C4 0.98 mm to (257.0, 176.5)
- moved C11 0.83 mm to (177.8, 177.2)
- moved D22 0.79 mm to (253.2, 185.8)
- moved C6 0.75 mm to (205.2, 173.0)
- moved C7 0.75 mm to (201.0, 177.5)
- moved C8 0.75 mm to (205.2, 176.0)
- moved R4 0.75 mm to (202.8, 170.0)
- moved R5 0.75 mm to (201.2, 170.0), turned to 90 degrees
- moved R6 0.75 mm to (199.8, 170.0)
- moved U1 0.75 mm to (202.8, 174.5)
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Connections:
- R5 pad 1: GND -> Net-(U1-ILIM/VSET)
- R5 pad 2: Net-(U1-ILIM/VSET) -> GND
- U1 pad 11: (no net) -> GND
- U2 pad 26: /CH_LED -> unconnected-(U2-P0.20-Pad26)
Routing:
- net VBUS: track 193.8 -> 164.2 mm, vias 6 -> 7
- net Net-(LED20-K): track 77.2 -> 60.4 mm
- net VDD: track 17.2 -> 25.6 mm
- net /SWDIO: track 17.1 -> 25.3 mm
- net /LED_PWM: track 139.4 -> 132.7 mm
- net +BATT: track 18.9 -> 13.2 mm
- net /LED_IN: track 104.3 -> 98.7 mm
- net /P10: track 71.9 -> 76.6 mm
- net /P2: track 169.6 -> 165.6 mm
- net /P7: track 197.3 -> 201.3 mm
- net /STAT1: track 109.5 -> 105.9 mm
- net /D+: track 65.0 -> 68.2 mm
- net /RESET: track 21.1 -> 24.2 mm
- net /STAT2: track 108.3 -> 105.4 mm
- net /D-: track 65.5 -> 68.3 mm
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- added copper zone on B.Cu, net GND
- added copper zone on F.Cu, net GND
Other:
- board size 147.6 x 103.5 mm -> 146.7 x 103.5 mm
- board text added: "CH"

Commit message: Preparation of mirror
Parts:
- S1, S10, S11, S12, S13, S14, S15, S16, S17, S18, S19, S2, S20, S21, S22, S3, S4, S5, S6, S7, S8, S9: footprint ceoloide:switch_gateron_ks27_ks33 -> ocdmk:switch_gateron_ks27_ks33
Connections:
- net /CH_LED renamed /Untitled Sheet/CH_LED
- net /D+ renamed /Untitled Sheet/D+
- net /D- renamed /Untitled Sheet/D-
- net /LED_IN renamed /Untitled Sheet/LED_IN
- net /LED_OUT renamed /Untitled Sheet/LED_OUT
- net /LED_PWM renamed /Untitled Sheet/LED_PWM
- net /P1 renamed /Untitled Sheet/P1
- net /P10 renamed /Untitled Sheet/P10
- net /P12 renamed /Untitled Sheet/P12
- net /P2 renamed /Untitled Sheet/P2
- net /P3 renamed /Untitled Sheet/P3
- net /P4 renamed /Untitled Sheet/P4
- net /P5 renamed /Untitled Sheet/P5
- net /P6 renamed /Untitled Sheet/P6
- net /P7 renamed /Untitled Sheet/P7
- net /P8 renamed /Untitled Sheet/P8
- net /P9 renamed /Untitled Sheet/P9
- net /RESET renamed /Untitled Sheet/RESET
- net /STAT1 renamed /Untitled Sheet/STAT1
- net /STAT2 renamed /Untitled Sheet/STAT2
- net /SWCLK renamed /Untitled Sheet/SWCLK
- net /SWDIO renamed /Untitled Sheet/SWDIO
- net /UART_RX renamed /Untitled Sheet/UART_RX
- net /UART_TX renamed /Untitled Sheet/UART_TX
