File: pcb/ocdmk.kicad_sch (KiCad schematic)
At the start: 101 parts, among them J1 USB_C_Receptacle_USB2.0_16P, J2 Conn_02x05_Odd_Even, J3 Conn_ARM_SWD_TagConnect_TC203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, J4 USB_C_Receptacle_USB2.0_16P, J5 Conn_01x02_Pin, SW1 SW_Push, U2 MDBT50-512K, U3 MCP1662-xOT

Commit message: Added components
Parts:
- removed C2: 100n, Capacitor_SMD:C_0603_1608Metric, symbol Device:C
- removed R1: 10k, Resistor_SMD:R_0603_1608Metric, symbol Device:R
- removed SW1: SW_Push, ceoloide:switch_gateron_ks27_ks33, symbol Switch:SW_Push
- C11: footprint Capacitor_SMD:C_0603_1608Metric -> Capacitor_SMD:C_1206_3216Metric
- JP1: footprint Resistor_SMD:R_0603_1608Metric -> Jumper:SolderJumper-2_P1.3mm_Open_TrianglePad1.0x1.5mm
- L3: value 4u7 -> 10u
- U1: value ~ -> bq25185
Connections:
- net GND: now also R5.2; no longer R5.1
- net at U1.7 (ILIM/VSET): now also R5.1; no longer R5.2
Other:
- note added: "R_{8} = 300mA/I_{SET} (current through diodes)"
- moved on the sheet: R4, R5

Commit message: half completed
Parts:
- removed J2: Conn_02x05_Odd_Even, symbol Connector_Generic:Conn_02x05_Odd_Even
- J1, J4: footprint ocdmk:USB4510-03-1-A_GCT -> ocdmk:12402012E212A_AMP
- J3: footprint Connector:Tag-Connect_TC2030-IDC-NL_2x03_P1.27mm_Vertical -> Connector:Tag-Connect_TC2030-IDC-FP_2x03_P1.27mm_Vertical
- J5: footprint Connector_JST:JST_PH_S2B-PH-SM4-TB_1x02-1MP_P2.00mm_Horizontal -> Connector_JST:JST_PH_S2B-PH-K_1x02_P2.00mm_Horizontal
Connections:
- net CH_LED: no longer U2.26 (P0.20)
- net GND: now also J1.S1 (SHIELD), J4.S1 (SHIELD), U1.11 (GND)

Commit message: Preparation of mirror
Parts:
- removed C1, C3, C6, C7: 1u, Capacitor_SMD:C_0603_1608Metric, symbol Device:C
- removed C11: 10u, Capacitor_SMD:C_1206_3216Metric, symbol Device:C
- removed C4, C5, C8: 10u, Capacitor_SMD:C_0603_1608Metric, symbol Device:C
- removed C9: 4u7, Capacitor_SMD:C_0603_1608Metric, symbol Device:C
- removed D1, D10, D11, D12, D13, D14, D15, D16, D17, D18, D19, D2, D20, D21, D22, D3, D4, D5, D6, D7, D8, D9: D, Diode_SMD:D_SOD-123, symbol Device:D
- removed D30: D_Schottky, Diode_SMD:D_SOD-123, symbol Device:D_Schottky
- removed J1, J4: USB_C_Receptacle_USB2.0_16P, ocdmk:12402012E212A_AMP, symbol Connector:USB_C_Receptacle_USB2.0_16P
- removed J3: Conn_ARM_SWD_TagConnect_TC2030-NL, Connector:Tag-Connect_TC2030-IDC-FP_2x03_P1.27mm_Vertical, symbol Connector:Conn_ARM_SWD_TagConnect_TC2030-NL
- removed J5: Conn_01x02_Pin, Connector_JST:JST_PH_S2B-PH-K_1x02_P2.00mm_Horizontal, symbol Connector:Conn_01x02_Pin
- removed JP1: Jumper_2_Open, Jumper:SolderJumper-2_P1.3mm_Open_TrianglePad1.0x1.5mm, symbol Jumper:Jumper_2_Open
- removed L1: 10u, Inductor_SMD:L_0805_2012Metric, symbol Device:L
- removed L2: 15n, Inductor_SMD:L_0603_1608Metric, symbol Device:L
- removed L3: 10u, Inductor_SMD:L_0603_1608Metric, symbol Device:L
- removed LED1, LED10, LED11, LED12, LED13, LED14, LED15, LED16, LED17, LED18, LED19, LED2, LED20, LED21, LED22, LED3, LED4, LED5, LED6, LED7, LED8, LED9: LED, ocdmk:LED_MP-2016-1100-50-90, symbol Device:LED
- removed LED23: LED, LED_SMD:LED_0603_1608Metric, symbol Device:LED
- removed R10, R7, R8, R9: 10, Resistor_SMD:R_0603_1608Metric, symbol Device:R
- removed R2, R3: 5.1k, Resistor_SMD:R_0603_1608Metric, symbol Device:R
- removed R4: 1k, Resistor_SMD:R_0603_1608Metric, symbol Device:R
- removed R5: 18k, Resistor_SMD:R_0603_1608Metric, symbol Device:R
- removed R6: 10k, Resistor_SMD:R_0603_1608Metric, symbol Device:R
- removed S1, S10, S11, S12, S13, S14, S15, S16, S17, S18, S19, S2, S20, S21, S22, S3, S4, S5, S6, S7, S8, S9: SW_Push, ceoloide:switch_gateron_ks27_ks33, symbol Switch:SW_Push
- removed U1: bq25185, ocdmk:SON50P250X250X80-11N, symbol ocdmk:BQ25185
- removed U2: MDBT50-512K, ocdmk:XCVR_MDBT50-512K, symbol MDBT50:MDBT50-512K
- removed U3: MCP1662-xOT, Package_TO_SOT_SMD:SOT-23-5, symbol Driver_LED:MCP1662-xOT
Other:
- added sheet Untitled Sheet (half.kicad_sch)
- note removed: "R_{8} = 300mA/I_{SET} (current through diodes)"
