File: pcb/core/core.kicad_sch (KiCad schematic)
At the start: 25 parts, among them J1 Conn_01x10, J2 Conn_01x07, J3 Conn_ARM_SWD_TagConnect_TC203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, J4 Conn_01x10, U1 bq25185, U2 MDBT50-512K, U3 MCP1662-xOT

Commit message: Some fixes on PCB
Parts:
- removed J3: Conn_ARM_SWD_TagConnect_TC2030-NL, Connector:Tag-Connect_TC2030-IDC-NL_2x03_P1.27mm_Vertical, symbol Connector:Conn_ARM_SWD_TagConnect_TC2030-NL
- added J6: Conn_02x05_Odd_Even, Connector_PinHeader_1.27mm:PinHeader_2x05_P1.27mm_Vertical, symbol Connector_Generic:Conn_02x05_Odd_Even
- L3: footprint Inductor_SMD:L_0805_2012Metric -> Inductor_SMD:L_0603_1608Metric
Connections:
- net GND: now also J6.3 (Pin_3), J6.5 (Pin_5)
- net RESET: now also J6.10 (Pin_10)
- net SWCLK: now also J6.4 (Pin_4)
- net SWDIO: now also J6.2 (Pin_2)
- net VDD: now also J6.1 (Pin_1)
