File: pcb/left/left_ocdmk.kicad_pcb (KiCad board)
At the start: 2 copper layers, 147.9 x 103.5 mm, 101 parts, among them J1 Conn_01x02

Commit message: Saved
Parts:
- removed D23, D24: LED, Diode_SMD:D_0603_1608Metric
- removed R1: 5.1k, Resistor_SMD:R_0603_1608Metric
- removed U2, U3: ~, Package_TO_SOT_SMD:SOT-553
- added REF**: SOT-363_SC-70-6, Package_TO_SOT_SMD:SOT-363_SC-70-6, F.Cu at (140.1, -9.26)
Connections:
- U1 pad 1: /LED -> unconnected-(U1-P0.15-Pad1)
Routing:
- net VBUS: track 87.9 -> 71.3 mm, vias 3 -> 4
- net Net-(D23-A): track 6.67 -> 0.00 mm, vias 2 -> 0
- net /LED: track 3.83 -> 0.00 mm
- net /UART_RX: track 35.7 -> 38.0 mm
- net /D+: track 9.35 -> 7.64 mm
- net /D-: track 15.5 -> 13.9 mm
- net GND: track 8.48 -> 7.39 mm, vias 133 -> 130
- net /UART_TX: track 39.7 -> 38.8 mm, vias 1 -> 0

Commit message: Some fixes on PCB
Parts:
- removed REF**: SOT-363_SC-70-6, Package_TO_SOT_SMD:SOT-363_SC-70-6
- added D23: LED, Diode_SMD:D_0603_1608Metric, F.Cu at (117.7, -59.8)
- added D24: LED, Diode_SMD:D_0603_1608Metric, B.Cu at (117.7, -59.8)
- added R1: 5.1k, Resistor_SMD:R_0603_1608Metric, F.Cu at (114.9, -55.2)
- added U2: ~, Package_TO_SOT_SMD:SOT-553, B.Cu at (126.3, -50.5)
- added U3: ~, Package_TO_SOT_SMD:SOT-553, F.Cu at (126.7, -13.3)
- added U4: ~, Package_TO_SOT_SMD:SOT-553, B.Cu at (126.7, -13.3)
- R2, R3, USB1: moved to B.Cu
- moved R2 12.8 mm to (119.5, -54.2)
- moved R3 12.7 mm to (132.0, -51.5)
- turned USB1 to -12.5 degrees
Connections:
- U1 pad 1: unconnected-(U1-P0.15-Pad1) -> /LED
Routing:
- net VBUS: track 71.3 -> 93.2 mm, vias 4 -> 5
- net Net-(D8-K): track 6.98 -> 15.5 mm
- net GND: track 7.39 -> 15.5 mm, vias 130 -> 146
- net Net-(D12-K): track 8.61 -> 15.8 mm
- net Net-(D11-K): track 8.82 -> 15.8 mm
- net Net-(D23-A): track 0.00 -> 6.67 mm, vias 0 -> 2
- net Net-(LEDB18-K): track 24.7 -> 29.3 mm, vias 1 -> 2
- net Net-(D18-K): track 5.44 -> 9.55 mm
- net /LED_A: track 157.6 -> 161.6 mm, vias 2 -> 4
- net /LED: track 0.00 -> 3.83 mm
- net /R2: track 151.7 -> 154.6 mm
- net /R3: track 166.7 -> 169.6 mm, vias 6 -> 7
- net /LED_K: track 57.9 -> 60.6 mm, vias 2 -> 3
- net /UART_TX: track 38.8 -> 41.5 mm, vias 0 -> 1
- net /UART_RX: track 38.0 -> 39.0 mm
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Other:
- board text added: "oCDMK v1.0"
